Commit message: edits to robot models, minimal controller and new gazebo doc

File: minimal_robot_description/minimal_robot_description.urdf (robot description, URDF)
Before this commit: robot one_link_robot, 3 links, 2 joints
Links:
- link link2: geometry collision cylinder length=1 radius=0.1; visual cylinder length=1 radius=0.1
Joints:
- removed joint fixed
- added joint glue_robot_to_world: type fixed, parent world, child link1
